File: Hardware/ARDUINO_8stepSeqV1_Schematic_Rev 2.0/ARDUINO_8stepSeqV1_Schematic.kicad_sch (KiCad schematic)
At the start: 20 parts, among them J1 AudioJack3, SW1 SW_Push, SW10 SW_Push, SW12 RotaryEncoder_Switch, SW2 SW_Push, SW3 SW_Push, SW4 SW_Push, SW5 SW_Push, SW6 SW_Push, SW7 SW_Push, SW8 SW_Push, SW9 SW_Push, U1 ER_OLEDM0.91_1x-I2C

Commit message: temp changes
Parts:
- removed A1: Arduino_Nano_v3.x, Module:Arduino_Nano, symbol MCU_Module:Arduino_Nano_v3.x
- added U2: ATmega328P-A, Package_QFP:TQFP-32_7x7mm_P0.8mm, symbol MCU_Microchip_ATmega:ATmega328P-A
- added Y1: 16Mhz, symbol Device:Crystal
Connections:
- new net: U2.21 (GND), U2.3 (GND), U2.5 (GND)
- new net: U2.4 (VCC), U2.6 (VCC)
- new net: U2.7 (XTAL1/PB6), Y1.2
- new net: U2.8 (XTAL2/PB7), Y1.1
Changed lines of the file:
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@@
 	(title_block
 		(title "Arduino Nano 8 step sequencer")
-		(date "2026-06-20")
-		(rev "V1.0")
+		(date "2026-07-03")
+		(rev "V2.0")
 		(company "Volquete Synth")
 		(comment 1 "Autor: Joan Benito Britez")
@@
 	(wire
 		(pts
+			(xy 260.35 80.01) (xy 270.51 80.01)
+		)
+		(stroke
+			(width 0)
+			(type default)
+		)
+	)
+	(wire
+		(pts
 			(xy 134.62 147.32) (xy 173.99 147.32)
 		)
@@
 	(wire
 		(pts
+			(xy 260.35 72.39) (xy 270.51 72.39)
+		)
+		(stroke
+			(width 0)
+			(type default)
+		)
+	)
+	(wire
+		(pts
 			(xy 36.83 130.81) (xy 36.83 139.7)
 		)
@@
 	(wire
 		(pts
+			(xy 254 74.93) (xy 260.35 74.93)
+		)
+		(stroke
+			(width 0)
+			(type default)
+		)
+	)
+	(wire
+		(pts
 			(xy 69.85 139.7) (xy 69.85 147.32)
 		)
@@
 	(wire
 		(pts
+			(xy 260.35 74.93) (xy 260.35 72.39)
+		)
+		(stroke
+			(width 0)
+			(type default)
+		)
+	)
+	(wire
+		(pts
 			(xy 200.66 72.39) (xy 200.66 80.01)
 		)
@@
 	(wire
 		(pts
+			(xy 260.35 77.47) (xy 260.35 80.01)
+		)
+		(stroke
+			(width 0)
+			(type default)
+		)
+	)
+	(wire
+		(pts
 			(xy 118.11 125.73) (xy 118.11 111.76)
 		)
@@
 		(pts
 			(xy 53.34 50.8) (xy 53.34 62.23)
+		)
+		(stroke
+			(width 0)
+			(type default)
+		)
+	)
+	(wire
+		(pts
+			(xy 254 77.47) (xy 260.35 77.47)
 		)
 		(stroke
@@
 	)
 	(symbol
+		(lib_id "MCU_Microchip_ATmega:ATmega328P-A")
+		(at 238.76 90.17 0)
+		(unit 1)
+		(body_style 1)
+		(exclude_from_sim no)
+		(in_bom yes)
+		(on_board yes)
+		(in_pos_files yes)
+		(dnp no)
+		(fields_autoplaced yes)
+		(property "Reference" "U2"
+			(at 240.9033 128.27 0)
+			(show_name no)
+			(do_not_autoplace no)
+			(effects
+				(font
+					(size 1.27 1.27)
+				)
+				(justify left)
+			)
+		)
+		(property "Value" "ATmega328P-A"
+			(at 240.9033 130.81 0)
+			(show_name no)
+			(do_not_autoplace no)
+			(effects
+				(font
+					(size 1.27 1.27)
+				)
+				(justify left)
+			)
+		)
+		(property "Footprint" "Package_QFP:TQFP-32_7x7mm_P0.8mm"
+			(at 238.76 90.17 0)
+			(show_name yes)
+			(do_not_autoplace no)
+			(effects
+				(font
+					(size 1.27 1.27)
+					(italic yes)
+				)
+			)
+		)
+		(property "Datasheet" "http://ww1.microchip.com/downloads/en/DeviceDoc/ATmega328_P%20AVR%20MCU%20with%20picoPower%20Technology%20Data%20Sheet%2040001984A.pdf"
+			(at 238.76 90.17 0)
+			(hide yes)
+			(show_name no)
+			(do_not_autoplace no)
+			(effects
+				(font
+					(size 1.27 1.27)
+				)
+			)
+		)
+		(property "Description" "20MHz, 32kB Flash, 2kB SRAM, 1kB EEPROM, TQFP-32"
+			(at 238.76 90.17 0)
+			(hide yes)
+			(show_name no)
+			(do_not_autoplace no)
+			(effects
+				(font
+					(size 1.27 1.27)
+				)
+			)
+		)
+		(pin "17"
+		)
+		(pin "3"
+		)
+		(pin "11"
+		)
+		(pin "25"
+		)
+		(pin "27"
+		)
+		(pin "13"
+		)
+		(pin "5"
+		)
+		(pin "20"
+		)
+		(pin "29"
+		)
+		(pin "22"
+		)
+		(pin "16"
+		)
+		(pin "23"
+		)
+		(pin "8"
+		)
+		(pin "14"
+		)
+		(pin "28"
+		)
+		(pin "30"
+		)
+		(pin "10"
+		)
+		(pin "31"
+		)
+		(pin "4"
+		)
+		(pin "7"
+		)
+		(pin "15"
+		)
+		(pin "19"
+		)
+		(pin "12"
+		)
+		(pin "26"
+		)
+		(pin "2"
+		)
+		(pin "24"
+		)
+		(pin "6"
+		)
+		(pin "9"
+		)
+		(pin "21"
+		)
+		(pin "32"
+		)
+		(pin "1"
+		)
+		(pin "18"
+		)
+		(instances
+			(project "ARDUINO_8stepSeqV1_Schematic"
+				(path "/6e0a64ec-f14f-4854-ab94-c7b052555216"
+					(reference "U2")
+					(unit 1)
+				)
+			)
+		)
+	)
+	(symbol
 		(lib_id "Device:R")
 		(at 116.84 57.15 0)
@@
 	)
 	(symbol
-		(lib_id "MCU_Module:Arduino_Nano_v3.x")
-		(at 134.62 93.98 0)
+		(lib_id "Device:Crystal")
+		(at 270.51 76.2 90)
 		(unit 1)
 		(body_style 1)
@@
 		(dnp no)
 		(fields_autoplaced yes)
-		(property "Reference" "A1"
-			(at 139.3033 119.38 0)
-			(show_name no)
-			(do_not_autoplace no)
-			(effects
-				(font
-					(size 1.27 1.27)
-				)
-				(justify left)
-			)
-		)
-		(property "Value" "Arduino_Nano_v3.x"
-			(at 139.3033 121.92 0)
-			(show_name no)
-			(do_not_autoplace no)
-			(effects
-				(font
-					(size 1.27 1.27)
-				)
-				(justify left)
-			)
-		)
-		(property "Footprint" "Module:Arduino_Nano"
-			(at 134.62 93.98 0)
-			(hide yes)
-			(show_name no)
-			(do_not_autoplace no)
-			(effects
-				(font
-					(size 1.27 1.27)
-					(italic yes)
-				)
-			)
-		)
-		(property "Datasheet" "http://www.mouser.com/pdfdocs/Gravitech_Arduino_Nano3_0.pdf"
-			(at 134.62 93.98 0)
-			(hide yes)
-			(show_name no)
-			(do_not_autoplace no)
-			(effects
-				(font
-					(size 1.27 1.27)
-				)
-			)
-		)
-		(property "Description" "Arduino Nano v3.x"
-			(at 134.62 93.98 0)
-			(hide yes)
-			(show_name no)
-			(do_not_autoplace no)
-			(effects
-				(font
-					(size 1.27 1.27)
-				)
-			)
-		)
-		(pin "8"
-		)
-		(pin "14"
-		)
-		(pin "22"
-		)
-		(pin "25"
-		)
-		(pin "5"
-		)
-		(pin "12"
-		)
-		(pin "16"
-		)
-		(pin "21"
-		)
-		(pin "6"
-		)
-		(pin "29"
-		)
-		(pin "4"
-		)
-		(pin "24"
+		(property "Reference" "Y1"
+			(at 274.32 74.9299 90)
+			(show_name no)
+			(do_not_autoplace no)
+			(effects
+				(font
+					(size 1.27 1.27)
+				)
+				(justify right)
+			)
+		)
+		(property "Value" "16Mhz"
+			(at 274.32 77.4699 90)
+			(show_name no)
+			(do_not_autoplace no)
+			(effects
+				(font
+					(size 1.27 1.27)
+				)
+				(justify right)
+			)
+		)
+		(property "Footprint" ""
+			(at 270.51 76.2 0)
+			(hide yes)
+			(show_name no)
+			(do_not_autoplace no)
+			(effects
+				(font
+					(size 1.27 1.27)
+				)
+			)
+		)
+		(property "Datasheet" ""
+			(at 270.51 76.2 0)
+			(hide yes)
+			(show_name no)
+			(do_not_autoplace no)
+			(effects
+				(font
+					(size 1.27 1.27)
+				)
+			)
+		)
+		(property "Description" "Two pin crystal"
+			(at 270.51 76.2 0)
+			(hide yes)
+			(show_name no)
+			(do_not_autoplace no)
+			(effects
+				(font
+					(size 1.27 1.27)
+				)
+			)
+		)
+		(pin "2"
 		)
 		(pin "1"
-		)
-		(pin "2"
-		)
-		(pin "3"
-		)
-		(pin "11"
-		)
-		(pin "10"
-		)
-		(pin "13"
-		)
-		(pin "17"
-		)
-		(pin "7"
-		)
-		(pin "9"
-		)
-		(pin "15"
-		)
-		(pin "18"
-		)
-		(pin "19"
-		)
-		(pin "20"
-		)
-		(pin "23"
-		)
-		(pin "26"
-		)
-		(pin "27"
-		)
-		(pin "28"
-		)
-		(pin "30"
 		)
 		(instances
 			(project "ARDUINO_8stepSeqV1_Schematic"
 				(path "/6e0a64ec-f14f-4854-ab94-c7b052555216"
-					(reference "A1")
+					(reference "Y1")
 					(unit 1)
 				)
